File: keyboard/keyboard.kicad_sch (KiCad schematic)
At the start: 0 parts

Commit message: 1.1
Parts:
- added J1: 5V, symbol Connector:Conn_01x02_Pin
- added SW1: SW_Push, symbol Switch:SW_Push
- added U1: ATmega328-P, Package_DIP:DIP-28_W7.62mm, symbol MCU_Microchip_ATmega:ATmega328-P
Connections:
- new net: U1.22 (GND), U1.8 (GND)
- new net +5V: J1.1 (Pin_1), SW1.2

Commit message: 1.1.0
Parts:
- removed J1: 5V, symbol Connector:Conn_01x02_Pin
- removed U1: ATmega328-P, Package_DIP:DIP-28_W7.62mm, symbol MCU_Microchip_ATmega:ATmega328-P
- added D1, D10, D100, D101, D102, D103, D104, D105, D106, D107, D108, D109, D11, D110, D111, D112, D113, D114, D115, D116, D117, D118, D119, D12, D120, D121, D122, D123, D124, D125, D126, D127, D128, D129, D13, D130, D131, D132, D133, D134, D135, D136, D137, D138, D139, D14, D140, D141, D142, D143, D144, D145, D146, D147, D148, D149, D15, D150, D151, D152, D153, D154, D155, D156, D157, D158, D159, D16, D17, D18, D19, D2, D20, D21, D22, D23, D24, D25, D26, D27, D28, D29, D3, D30, D31, D32, D33, D34, D35, D36, D37, D38, D39, D4, D40, D41, D42, D43, D44, D45, D46, D47, D48, D49, D5, D50, D51, D52, D53, D54, D55, D56, D57, D58, D59, D6, D60, D61, D62, D63, D64, D65, D66, D67, D68, D69, D7, D70, D71, D72, D73, D74, D75, D76, D77, D78, D79, D8, D80, D81, D82, D83, D84, D85, D86, D87, D88, D89, D9, D90, D91, D92, D93, D94, D95, D96, D97, D98, D99: D, Diode_THT:D_DO-41_SOD81_P7.62mm_Horizontal, symbol Device:D
- added J1: 5V in, Connector_Molex:Molex_CLIK-Mate_502382-1570_1x15-1MP_P1.25mm_Vertical, symbol Connector:Conn_01x02_Socket
- added R1, R10, R11, R12, R13, R14, R15, R16, R17, R2, R3, R4, R5, R6, R7, R8, R9: 10kΩ, Resistor_THT:R_Axial_DIN0411_L9.9mm_D3.6mm_P12.70mm_Horizontal, symbol Device:R
- added SW10: 0, Button_Switch_THT:SW_PUSH_6mm_H4.3mm, symbol Switch:SW_Push
- added SW11: ESC, Button_Switch_THT:SW_PUSH_6mm_H4.3mm, symbol Switch:SW_Push
- added SW12: Q, Button_Switch_THT:SW_PUSH_6mm_H4.3mm, symbol Switch:SW_Push
- added SW13: W, Button_Switch_THT:SW_PUSH_6mm_H4.3mm, symbol Switch:SW_Push
- added SW14: E, Button_Switch_THT:SW_PUSH_6mm_H4.3mm, symbol Switch:SW_Push
- added SW15: R, Button_Switch_THT:SW_PUSH_6mm_H4.3mm, symbol Switch:SW_Push
- added SW16: T, Button_Switch_THT:SW_PUSH_6mm_H4.3mm, symbol Switch:SW_Push
- added SW17: Y, Button_Switch_THT:SW_PUSH_6mm_H4.3mm, symbol Switch:SW_Push
- added SW18: U, Button_Switch_THT:SW_PUSH_6mm_H4.3mm, symbol Switch:SW_Push
- added SW19: I, Button_Switch_THT:SW_PUSH_6mm_H4.3mm, symbol Switch:SW_Push
- added SW2: 2, Button_Switch_THT:SW_PUSH_6mm_H4.3mm, symbol Switch:SW_Push
- added SW20: O, Button_Switch_THT:SW_PUSH_6mm_H4.3mm, symbol Switch:SW_Push
- added SW21: P, Button_Switch_THT:SW_PUSH_6mm_H4.3mm, symbol Switch:SW_Push
- added SW22: TAB, Button_Switch_THT:SW_PUSH_6mm_H4.3mm, symbol Switch:SW_Push
- added SW23: A, Button_Switch_THT:SW_PUSH_6mm_H4.3mm, symbol Switch:SW_Push
- added SW24: S, Button_Switch_THT:SW_PUSH_6mm_H4.3mm, symbol Switch:SW_Push
- added SW25: D, Button_Switch_THT:SW_PUSH_6mm_H4.3mm, symbol Switch:SW_Push
- added SW26: F, Button_Switch_THT:SW_PUSH_6mm_H4.3mm, symbol Switch:SW_Push
- added SW27: G, Button_Switch_THT:SW_PUSH_6mm_H4.3mm, symbol Switch:SW_Push
- added SW28: H, Button_Switch_THT:SW_PUSH_6mm_H4.3mm, symbol Switch:SW_Push
- added SW29: J, Button_Switch_THT:SW_PUSH_6mm_H4.3mm, symbol Switch:SW_Push
- added SW3: 3, Button_Switch_THT:SW_PUSH_6mm_H4.3mm, symbol Switch:SW_Push
- added SW30: K, Button_Switch_THT:SW_PUSH_6mm_H4.3mm, symbol Switch:SW_Push
- added SW31: L, Button_Switch_THT:SW_PUSH_6mm_H4.3mm, symbol Switch:SW_Push
- added SW32: '*, Button_Switch_THT:SW_PUSH_6mm_H4.3mm, symbol Switch:SW_Push
- added SW33: SHIFT, Button_Switch_THT:SW_PUSH_6mm_H4.3mm, symbol Switch:SW_Push
- added SW34: <|>, Button_Switch_THT:SW_PUSH_6mm_H4.3mm, symbol Switch:SW_Push
- added SW35: Z, Button_Switch_THT:SW_PUSH_6mm_H4.3mm, symbol Switch:SW_Push
- added SW36: X, Button_Switch_THT:SW_PUSH_6mm_H4.3mm, symbol Switch:SW_Push
- added SW37: C, Button_Switch_THT:SW_PUSH_6mm_H4.3mm, symbol Switch:SW_Push
- added SW38: V, Button_Switch_THT:SW_PUSH_6mm_H4.3mm, symbol Switch:SW_Push
- added SW39: B, Button_Switch_THT:SW_PUSH_6mm_H4.3mm, symbol Switch:SW_Push
- added SW4: 4, Button_Switch_THT:SW_PUSH_6mm_H4.3mm, symbol Switch:SW_Push
- added SW40: N, Button_Switch_THT:SW_PUSH_6mm_H4.3mm, symbol Switch:SW_Push
- added SW41: M, Button_Switch_THT:SW_PUSH_6mm_H4.3mm, symbol Switch:SW_Push
- added SW42: ,;, Button_Switch_THT:SW_PUSH_6mm_H4.3mm, symbol Switch:SW_Push
- added SW43: .:, Button_Switch_THT:SW_PUSH_6mm_H4.3mm, symbol Switch:SW_Push
- added SW44: CTRL, Button_Switch_THT:SW_PUSH_6mm_H4.3mm, symbol Switch:SW_Push
- added SW45: SPACE, Button_Switch_THT:SW_PUSH_6mm_H4.3mm, symbol Switch:SW_Push
- added SW46: ALTGR, Button_Switch_THT:SW_PUSH_6mm_H4.3mm, symbol Switch:SW_Push
- added SW47: RETURN, Button_Switch_THT:SW_PUSH_6mm_H4.3mm, symbol Switch:SW_Push
- added SW48: ENTER, Button_Switch_THT:SW_PUSH_6mm_H4.3mm, symbol Switch:SW_Push
- added SW49: -_, Button_Switch_THT:SW_PUSH_6mm_H4.3mm, symbol Switch:SW_Push
- added SW5: 5, Button_Switch_THT:SW_PUSH_6mm_H4.3mm, symbol Switch:SW_Push
- added SW50: UP, Button_Switch_THT:SW_PUSH_6mm_H4.3mm, symbol Switch:SW_Push
- added SW51: RIGHT, Button_Switch_THT:SW_PUSH_6mm_H4.3mm, symbol Switch:SW_Push
- added SW52: DOWN, Button_Switch_THT:SW_PUSH_6mm_H4.3mm, symbol Switch:SW_Push
- added SW53: LEFT, Button_Switch_THT:SW_PUSH_6mm_H4.3mm, symbol Switch:SW_Push
- added SW6: 6, Button_Switch_THT:SW_PUSH_6mm_H4.3mm, symbol Switch:SW_Push
- added SW7: 7, Button_Switch_THT:SW_PUSH_6mm_H4.3mm, symbol Switch:SW_Push
- added SW8: 8, Button_Switch_THT:SW_PUSH_6mm_H4.3mm, symbol Switch:SW_Push
- added SW9: 9, Button_Switch_THT:SW_PUSH_6mm_H4.3mm, symbol Switch:SW_Push
- added U1: ATmega48-20P, Package_DIP:DIP-28_W7.62mm, symbol MCU_Microchip_ATmega:ATmega48-20P
- SW1: value SW_Push -> 1; footprint (none) -> Button_Switch_THT:SW_PUSH_6mm_H4.3mm
Connections:
- net +5V: now also SW1.1, J1.1 (Pin_1), SW10.1, SW11.1, SW12.1, SW13.1, SW14.1, SW15.1, SW16.1, SW17.1, SW18.1, SW19.1, SW2.1, SW20.1, SW21.1, SW22.1, SW23.1, SW24.1, SW25.1, SW26.1, SW27.1, SW28.1, SW29.1, SW3.1, SW30.1, SW31.1, SW32.1, SW33.1, SW34.1, SW35.1, SW36.1, SW37.1, SW38.1, SW39.1, SW4.1, SW40.1, SW41.1, SW42.1, SW43.1, SW44.1, SW45.1, SW46.1, SW47.1, SW48.1, SW49.1, SW5.1, SW50.1, SW51.1, SW52.1, SW53.1, SW6.1, SW7.1, SW8.1, SW9.1, U1.7 (VCC); no longer SW1.2
- net ROW1: now also D11.1 (K), D14.1 (K), D17.1 (K), D2.1 (K), D20.1 (K), D23.1 (K), D26.1 (K), D29.1 (K), D5.1 (K), D8.1 (K), R13.1, U1.2 (PD0)
- new net: D61.2 (A), D62.2 (A), D63.2 (A), SW21.2
- new net: D121.2 (A), D122.2 (A), D123.2 (A), SW41.2
- new net: D151.2 (A), D152.2 (A), D153.2 (A), SW51.2
- new net: D73.2 (A), D74.2 (A), D75.2 (A), SW25.2
- new net: D25.2 (A), D26.2 (A), D27.2 (A), SW9.2
- new net: D157.2 (A), D158.2 (A), D159.2 (A), SW53.2
- new net: D100.2 (A), D101.2 (A), D102.2 (A), SW34.2
- new net: D67.2 (A), D68.2 (A), D69.2 (A), SW23.2
- new net: D106.2 (A), D107.2 (A), D108.2 (A), SW36.2
- new net: D124.2 (A), D125.2 (A), D126.2 (A), SW42.2
- new net: D4.2 (A), D5.2 (A), D6.2 (A), SW2.2
- new net: D112.2 (A), D113.2 (A), D114.2 (A), SW38.2
- new net: D133.2 (A), D134.2 (A), D135.2 (A), SW45.2
- new net: D130.2 (A), D131.2 (A), D132.2 (A), SW44.2
- new net: D31.2 (A), D32.2 (A), D33.2 (A), SW11.2
- new net: D13.2 (A), D14.2 (A), D15.2 (A), SW5.2
- new net: D55.2 (A), D56.2 (A), D57.2 (A), SW19.2
- new net: D43.2 (A), D44.2 (A), D45.2 (A), SW15.2
- new net: D40.2 (A), D41.2 (A), D42.2 (A), SW14.2
- new net: D46.2 (A), D47.2 (A), D48.2 (A), SW16.2
- new net: D22.2 (A), D23.2 (A), D24.2 (A), SW8.2
- new net: D115.2 (A), D116.2 (A), D117.2 (A), SW39.2
- new net: D118.2 (A), D119.2 (A), D120.2 (A), SW40.2
- new net: D148.2 (A), D149.2 (A), D150.2 (A), SW50.2
- new net: D34.2 (A), D35.2 (A), D36.2 (A), SW12.2
- new net: D139.2 (A), D140.2 (A), D141.2 (A), SW47.2
- new net: D127.2 (A), D128.2 (A), D129.2 (A), SW43.2
- new net: D19.2 (A), D20.2 (A), D21.2 (A), SW7.2
- new net: D52.2 (A), D53.2 (A), D54.2 (A), SW18.2
- new net: D109.2 (A), D110.2 (A), D111.2 (A), SW37.2
- new net: D97.2 (A), D98.2 (A), D99.2 (A), SW33.2
- new net: D64.2 (A), D65.2 (A), D66.2 (A), SW22.2
- new net: D88.2 (A), D89.2 (A), D90.2 (A), SW30.2
- new net: D82.2 (A), D83.2 (A), D84.2 (A), SW28.2
- new net: D7.2 (A), D8.2 (A), D9.2 (A), SW3.2
- new net: D37.2 (A), D38.2 (A), D39.2 (A), SW13.2
- new net: D10.2 (A), D11.2 (A), D12.2 (A), SW4.2
- new net: D103.2 (A), D104.2 (A), D105.2 (A), SW35.2
- new net: D1.2 (A), D2.2 (A), D3.2 (A), SW1.2
- new net: D49.2 (A), D50.2 (A), D51.2 (A), SW17.2
- new net: D154.2 (A), D155.2 (A), D156.2 (A), SW52.2
- new net: D76.2 (A), D77.2 (A), D78.2 (A), SW26.2
- new net: D70.2 (A), D71.2 (A), D72.2 (A), SW24.2
- new net: D91.2 (A), D92.2 (A), D93.2 (A), SW31.2
- new net: D136.2 (A), D137.2 (A), D138.2 (A), SW46.2
- new net: D145.2 (A), D146.2 (A), D147.2 (A), SW49.2
- new net: D58.2 (A), D59.2 (A), D60.2 (A), SW20.2
- new net: D28.2 (A), D29.2 (A), D30.2 (A), SW10.2
- new net: D94.2 (A), D95.2 (A), D96.2 (A), SW32.2
- new net: D85.2 (A), D86.2 (A), D87.2 (A), SW29.2
- new net: D142.2 (A), D143.2 (A), D144.2 (A), SW48.2
- new net: D16.2 (A), D17.2 (A), D18.2 (A), SW6.2
- new net: D79.2 (A), D80.2 (A), D81.2 (A), SW27.2
- new net COL1: D1.1 (K), D130.1 (K), D31.1 (K), D64.1 (K), D97.1 (K), R2.1, U1.15 (PB1)
- new net COL10: D124.1 (K), D157.1 (K), D28.1 (K), D58.1 (K), D91.1 (K), R11.1, U1.27 (PC4)
- new net COL11: D127.1 (K), D61.1 (K), D94.1 (K), R12.1, U1.28 (PC5)
- new net COL2: D100.1 (K), D133.1 (K), D34.1 (K), D4.1 (K), D67.1 (K), R3.1, U1.16 (PB2)
- new net COL3: D103.1 (K), D136.1 (K), D37.1 (K), D7.1 (K), D70.1 (K), R4.1, U1.17 (PB3)
- new net COL4: D10.1 (K), D106.1 (K), D139.1 (K), D40.1 (K), D73.1 (K), R5.1, U1.18 (PB4)
- new net COL5: D109.1 (K), D13.1 (K), D142.1 (K), D43.1 (K), D76.1 (K), R6.1, U1.19 (PB5)
- new net COL6: D112.1 (K), D145.1 (K), D16.1 (K), D46.1 (K), D79.1 (K), R7.1, U1.23 (PC0)
- new net COL7: D115.1 (K), D148.1 (K), D19.1 (K), D49.1 (K), D82.1 (K), R8.1, U1.24 (PC1)
- new net COL8: D118.1 (K), D151.1 (K), D22.1 (K), D52.1 (K), D85.1 (K), R9.1, U1.25 (PC2)
- new net COL9: D121.1 (K), D154.1 (K), D25.1 (K), D55.1 (K), D88.1 (K), R10.1, U1.26 (PC3)
- new net Detection: D102.1 (K), D105.1 (K), D108.1 (K), D111.1 (K), D114.1 (K), D117.1 (K), D12.1 (K), D120.1 (K), D123.1 (K), D126.1 (K), D129.1 (K), D132.1 (K), D135.1 (K), D138.1 (K), D141.1 (K), D144.1 (K), D147.1 (K), D15.1 (K), D150.1 (K), D153.1 (K), D156.1 (K), D159.1 (K), D18.1 (K), D21.1 (K), D24.1 (K), D27.1 (K), D3.1 (K), D30.1 (K), D33.1 (K), D36.1 (K), D39.1 (K), D42.1 (K), D45.1 (K), D48.1 (K), D51.1 (K), D54.1 (K), D57.1 (K), D6.1 (K), D60.1 (K), D63.1 (K), D66.1 (K), D69.1 (K), D72.1 (K), D75.1 (K), D78.1 (K), D81.1 (K), D84.1 (K), D87.1 (K), D9.1 (K), D90.1 (K), D93.1 (K), D96.1 (K), D99.1 (K), R1.1, U1.14 (PB0)
- new net GND: J1.2 (Pin_2), R1.2, R10.2, R11.2, R12.2, R13.2, R14.2, R15.2, R16.2, R17.2, R2.2, R3.2, R4.2, R5.2, R6.2, R7.2, R8.2, R9.2, U1.22 (GND), U1.8 (GND)
- new net ROW2: D32.1 (K), D35.1 (K), D38.1 (K), D41.1 (K), D44.1 (K), D47.1 (K), D50.1 (K), D53.1 (K), D56.1 (K), D59.1 (K), D62.1 (K), R14.1, U1.3 (PD1)
- new net ROW3: D65.1 (K), D68.1 (K), D71.1 (K), D74.1 (K), D77.1 (K), D80.1 (K), D83.1 (K), D86.1 (K), D89.1 (K), D92.1 (K), D95.1 (K), R15.1, U1.4 (PD2)
- new net ROW4: D101.1 (K), D104.1 (K), D107.1 (K), D110.1 (K), D113.1 (K), D116.1 (K), D119.1 (K), D122.1 (K), D125.1 (K), D128.1 (K), D98.1 (K), R16.1, U1.5 (PD3)
- new net ROW5: D131.1 (K), D134.1 (K), D137.1 (K), D140.1 (K), D143.1 (K), D146.1 (K), D149.1 (K), D152.1 (K), D155.1 (K), D158.1 (K), R17.1, U1.6 (PD4)

Commit message: 1.1.0
Parts:
- removed D10, D100, D101, D102, D103, D104, D105, D106, D107, D108, D109, D11, D110, D111, D112, D113, D114, D115, D116, D117, D118, D119, D12, D120, D121, D122, D123, D124, D125, D126, D127, D128, D129, D13, D130, D131, D132, D133, D134, D135, D136, D137, D138, D139, D14, D140, D141, D142, D143, D144, D145, D146, D147, D148, D149, D15, D150, D151, D152, D153, D154, D155, D156, D157, D158, D159, D16, D17, D18, D19, D20, D21, D22, D23, D24, D25, D26, D27, D28, D29, D30, D31, D32, D33, D34, D35, D36, D37, D38, D39, D40, D41, D42, D43, D44, D45, D46, D47, D48, D49, D5, D50, D51, D52, D53, D54, D55, D56, D57, D58, D59, D6, D60, D61, D62, D63, D64, D65, D66, D67, D68, D69, D7, D70, D71, D72, D73, D74, D75, D76, D77, D78, D79, D8, D80, D81, D82, D83, D84, D85, D86, D87, D88, D89, D9, D90, D91, D92, D93, D94, D95, D96, D97, D98, D99: D, Diode_THT:D_DO-41_SOD81_P7.62mm_Horizontal, symbol Device:D
- removed R10, R11, R12, R13, R14, R15, R16, R17, R7, R8, R9: 10kΩ, Resistor_THT:R_Axial_DIN0411_L9.9mm_D3.6mm_P12.70mm_Horizontal, symbol Device:R
- removed SW43: .:, Button_Switch_THT:SW_PUSH_6mm_H4.3mm, symbol Switch:SW_Push
- removed SW44: CTRL, Button_Switch_THT:SW_PUSH_6mm_H4.3mm, symbol Switch:SW_Push
- removed SW45: SPACE, Button_Switch_THT:SW_PUSH_6mm_H4.3mm, symbol Switch:SW_Push
- removed SW46: ALTGR, Button_Switch_THT:SW_PUSH_6mm_H4.3mm, symbol Switch:SW_Push
- removed SW47: RETURN, Button_Switch_THT:SW_PUSH_6mm_H4.3mm, symbol Switch:SW_Push
- removed SW48: ENTER, Button_Switch_THT:SW_PUSH_6mm_H4.3mm, symbol Switch:SW_Push
- removed SW49: -_, Button_Switch_THT:SW_PUSH_6mm_H4.3mm, symbol Switch:SW_Push
- removed SW50: UP, Button_Switch_THT:SW_PUSH_6mm_H4.3mm, symbol Switch:SW_Push
- removed SW51: RIGHT, Button_Switch_THT:SW_PUSH_6mm_H4.3mm, symbol Switch:SW_Push
- removed SW52: DOWN, Button_Switch_THT:SW_PUSH_6mm_H4.3mm, symbol Switch:SW_Push
- removed SW53: LEFT, Button_Switch_THT:SW_PUSH_6mm_H4.3mm, symbol Switch:SW_Push
- added C1: C, symbol Device:C
- D1, D2, D3, D4: footprint Diode_THT:D_DO-41_SOD81_P7.62mm_Horizontal -> (none)
- J1: value 5V in -> Conn_01x02_Socket; footprint Connector_Molex:Molex_CLIK-Mate_502382-1570_1x15-1MP_P1.25mm_Vertical -> (none)
- R1, R2, R3, R4, R5, R6: value 10kΩ -> 10k; footprint Resistor_THT:R_Axial_DIN0411_L9.9mm_D3.6mm_P12.70mm_Horizontal -> (none)
- SW1: value 1 -> SW_Push; footprint Button_Switch_THT:SW_PUSH_6mm_H4.3mm -> (none)
- SW10: value 0 -> SW_Push; footprint Button_Switch_THT:SW_PUSH_6mm_H4.3mm -> (none)
- SW11: value ESC -> SW_Push; footprint Button_Switch_THT:SW_PUSH_6mm_H4.3mm -> (none)
- SW12: value Q -> SW_Push; footprint Button_Switch_THT:SW_PUSH_6mm_H4.3mm -> (none)
- SW13: value W -> SW_Push; footprint Button_Switch_THT:SW_PUSH_6mm_H4.3mm -> (none)
- SW14: value E -> SW_Push; footprint Button_Switch_THT:SW_PUSH_6mm_H4.3mm -> (none)
- SW15: value R -> SW_Push; footprint Button_Switch_THT:SW_PUSH_6mm_H4.3mm -> (none)
- SW16: value T -> SW_Push; footprint Button_Switch_THT:SW_PUSH_6mm_H4.3mm -> (none)
- SW17: value Y -> SW_Push; footprint Button_Switch_THT:SW_PUSH_6mm_H4.3mm -> (none)
- SW18: value U -> SW_Push; footprint Button_Switch_THT:SW_PUSH_6mm_H4.3mm -> (none)
- SW19: value I -> SW_Push; footprint Button_Switch_THT:SW_PUSH_6mm_H4.3mm -> (none)
- SW2: value 2 -> SW_Push; footprint Button_Switch_THT:SW_PUSH_6mm_H4.3mm -> (none)
- SW20: value O -> SW_Push; footprint Button_Switch_THT:SW_PUSH_6mm_H4.3mm -> (none)
- SW21: value P -> SW_Push; footprint Button_Switch_THT:SW_PUSH_6mm_H4.3mm -> (none)
- SW22: value TAB -> SW_Push; footprint Button_Switch_THT:SW_PUSH_6mm_H4.3mm -> (none)
- SW23: value A -> SW_Push; footprint Button_Switch_THT:SW_PUSH_6mm_H4.3mm -> (none)
- SW24: value S -> SW_Push; footprint Button_Switch_THT:SW_PUSH_6mm_H4.3mm -> (none)
- SW25: value D -> SW_Push; footprint Button_Switch_THT:SW_PUSH_6mm_H4.3mm -> (none)
- SW26: value F -> SW_Push; footprint Button_Switch_THT:SW_PUSH_6mm_H4.3mm -> (none)
- SW27: value G -> SW_Push; footprint Button_Switch_THT:SW_PUSH_6mm_H4.3mm -> (none)
- SW28: value H -> SW_Push; footprint Button_Switch_THT:SW_PUSH_6mm_H4.3mm -> (none)
- SW29: value J -> SW_Push; footprint Button_Switch_THT:SW_PUSH_6mm_H4.3mm -> (none)
- SW3: value 3 -> SW_Push; footprint Button_Switch_THT:SW_PUSH_6mm_H4.3mm -> (none)
- SW30: value K -> SW_Push; footprint Button_Switch_THT:SW_PUSH_6mm_H4.3mm -> (none)
- SW31: value L -> SW_Push; footprint Button_Switch_THT:SW_PUSH_6mm_H4.3mm -> (none)
- SW32: value '* -> SW_Push; footprint Button_Switch_THT:SW_PUSH_6mm_H4.3mm -> (none)
- SW33: value SHIFT -> SW_Push; footprint Button_Switch_THT:SW_PUSH_6mm_H4.3mm -> (none)
- SW34: value <|> -> SW_Push; footprint Button_Switch_THT:SW_PUSH_6mm_H4.3mm -> (none)
- SW35: value Z -> SW_Push; footprint Button_Switch_THT:SW_PUSH_6mm_H4.3mm -> (none)
- SW36: value X -> SW_Push; footprint Button_Switch_THT:SW_PUSH_6mm_H4.3mm -> (none)
- SW37: value C -> SW_Push; footprint Button_Switch_THT:SW_PUSH_6mm_H4.3mm -> (none)
- SW38: value V -> SW_Push; footprint Button_Switch_THT:SW_PUSH_6mm_H4.3mm -> (none)
- SW39: value B -> SW_Push; footprint Button_Switch_THT:SW_PUSH_6mm_H4.3mm -> (none)
- SW4: value 4 -> SW_Push; footprint Button_Switch_THT:SW_PUSH_6mm_H4.3mm -> (none)
- SW40: value N -> SW_Push; footprint Button_Switch_THT:SW_PUSH_6mm_H4.3mm -> (none)
- SW41: value M -> SW_Push; footprint Button_Switch_THT:SW_PUSH_6mm_H4.3mm -> (none)
- SW42: value ,; -> SW_Push; footprint Button_Switch_THT:SW_PUSH_6mm_H4.3mm -> (none)
- SW5: value 5 -> SW_Push; footprint Button_Switch_THT:SW_PUSH_6mm_H4.3mm -> (none)
- SW6: value 6 -> SW_Push; footprint Button_Switch_THT:SW_PUSH_6mm_H4.3mm -> (none)
- SW7: value 7 -> SW_Push; footprint Button_Switch_THT:SW_PUSH_6mm_H4.3mm -> (none)
- SW8: value 8 -> SW_Push; footprint Button_Switch_THT:SW_PUSH_6mm_H4.3mm -> (none)
- SW9: value 9 -> SW_Push; footprint Button_Switch_THT:SW_PUSH_6mm_H4.3mm -> (none)
Connections:
- net +5V: now also R6.2, U1.20 (AVCC); no longer SW1.1, SW10.1, SW11.1, SW12.1, SW13.1, SW14.1, SW15.1, SW16.1, SW17.1, SW18.1, SW19.1, SW2.1, SW20.1, SW21.1, SW22.1, SW23.1, SW24.1, SW25.1, SW26.1, SW27.1, SW28.1, SW29.1, SW3.1, SW30.1, SW31.1, SW32.1, SW33.1, SW34.1, SW35.1, SW36.1, SW37.1, SW38.1, SW39.1, SW4.1, SW40.1, SW41.1, SW42.1, SW5.1, SW6.1, SW7.1, SW8.1, SW9.1
- net COL1: now also SW1.2, SW12.2, SW23.2, SW34.2, U1.14 (PB0); no longer D1.1 (K), R2.1, U1.15 (PB1)
- net COL10: now also SW10.2, SW21.2, SW32.2, U1.24 (PC1); no longer U1.27 (PC4)
- net COL11: now also SW11.2, SW22.2, SW33.2, U1.25 (PC2); no longer U1.28 (PC5)
- net COL2: now also SW13.2, SW2.2, SW24.1, SW35.2, U1.15 (PB1); no longer D4.1 (K), R3.1, U1.16 (PB2)
- net COL3: now also SW14.2, SW25.2, SW3.2, SW36.2, U1.16 (PB2); no longer R4.1, U1.17 (PB3)
- net COL4: now also SW15.2, SW26.2, SW37.2, SW4.2, U1.17 (PB3); no longer R5.1, U1.18 (PB4)
- net COL5: now also SW16.2, SW27.2, SW38.2, SW5.2, U1.18 (PB4); no longer R6.1, U1.19 (PB5)
- net COL6: now also SW17.2, SW28.2, SW39.2, SW6.2, U1.19 (PB5); no longer U1.23 (PC0)
- net COL7: now also SW18.2, SW29.2, SW40.2, SW7.2, U1.9 (XTAL1/PB6); no longer U1.24 (PC1)
- net COL8: now also SW19.2, SW30.2, SW41.2, SW8.2, U1.10 (XTAL2/PB7); no longer U1.25 (PC2)
- net COL9: now also SW20.2, SW31.2, SW42.2, SW9.2, U1.23 (PC0); no longer U1.26 (PC3)
- net GND: now also R1.1, R2.1, R3.1, R4.1, R5.1, C1.2; no longer R1.2, R2.2, R3.2, R4.2, R5.2, R6.2
- net ROW1: now also D1.2 (A), R1.2, SW1.1, SW10.1, SW11.1, SW2.1, SW3.1, SW4.1, SW5.1, SW6.1, SW7.1, SW8.1, SW9.1, U1.26 (PC3); no longer D2.1 (K), U1.2 (PD0)
- net ROW2: now also D2.2 (A), R2.2, SW12.1, SW13.1, SW14.1, SW15.1, SW16.1, SW17.1, SW18.1, SW19.1, SW20.1, SW21.1, SW22.1, U1.27 (PC4); no longer U1.3 (PD1)
- net ROW3: now also D3.2 (A), R3.2, SW23.1, SW24.2, SW25.1, SW26.1, SW27.1, SW28.1, SW29.1, SW30.1, SW31.1, SW32.1, SW33.1, U1.28 (PC5); no longer U1.4 (PD2)
- net ROW4: now also D4.2 (A), R4.2, SW34.1, SW35.1, SW36.1, SW37.1, SW38.1, SW39.1, SW40.1, SW41.1, SW42.1, U1.2 (PD0); no longer U1.5 (PD3)
- net at U1.1 (~{RESET}/PC6): now also R6.1
- net at U1.21 (AREF): now also C1.1
- removed net Detection: D3.1 (K), R1.1, U1.14 (PB0)
- net ROW5: no longer names the net of U1.6 (PD4)
- new net Trigger: D1.1 (K), D2.1 (K), D3.1 (K), D4.1 (K), R5.2, U1.3 (PD1)
