File: keyboard/keyboard.kicad_sch (KiCad schematic)
At the start: 0 parts

Commit message: 1.5
Parts:
- added C1: C, Capacitor_THT:CP_Radial_D4.0mm_P2.00mm, symbol Device:C
- added D1, D2, D3, D4: D, Diode_THT:D_DO-41_SOD81_P7.62mm_Horizontal, symbol Device:D
- added J1: Conn_01x02_Socket, Connector_JST:JST_EH_S2B-EH_1x02_P2.50mm_Horizontal, symbol Connector:Conn_01x02_Socket
- added R1, R2, R3, R4, R5, R6: 10k, Resistor_THT:R_Axial_DIN0207_L6.3mm_D2.5mm_P7.62mm_Horizontal, symbol Device:R
- added SW1, SW10, SW11, SW12, SW13, SW14, SW15, SW16, SW17, SW18, SW19, SW2, SW20, SW21, SW22, SW23, SW24, SW25, SW26, SW27, SW28, SW29, SW3, SW30, SW31, SW32, SW33, SW34, SW35, SW36, SW37, SW38, SW39, SW4, SW40, SW41, SW42, SW5, SW6, SW7, SW8, SW9: SW_Push, Button_Switch_THT:SW_PUSH_6mm_H4.3mm, symbol Switch:SW_Push
- added U1: ATmega48-20P, Package_DIP:DIP-28_W7.62mm, symbol MCU_Microchip_ATmega:ATmega48-20P
Connections:
- new net: R6.1, U1.1 (~{RESET}/PC6)
- new net: C1.1, U1.21 (AREF)
- new net +5V: J1.1 (Pin_1), R6.2, U1.20 (AVCC), U1.7 (VCC)
- new net COL1: SW1.2, SW12.2, SW23.2, SW34.2, U1.14 (PB0)
- new net COL10: SW10.2, SW21.2, SW32.2, SW41.2, U1.24 (PC1)
- new net COL11: SW11.2, SW22.2, SW33.2, SW42.2, U1.25 (PC2)
- new net COL2: SW13.2, SW2.2, SW24.2, SW35.2, U1.15 (PB1)
- new net COL3: SW14.2, SW25.2, SW3.2, U1.16 (PB2)
- new net COL4: SW15.2, SW26.2, SW36.2, SW4.2, U1.17 (PB3)
- new net COL5: SW16.2, SW27.2, SW5.2, U1.18 (PB4)
- new net COL6: SW17.2, SW28.2, SW37.2, SW6.2, U1.19 (PB5)
- new net COL7: SW18.2, SW29.2, SW38.2, SW7.2, U1.9 (XTAL1/PB6)
- new net COL8: SW19.2, SW30.2, SW39.2, SW8.2, U1.10 (XTAL2/PB7)
- new net COL9: SW20.2, SW31.2, SW40.2, SW9.2, U1.23 (PC0)
- new net GND: C1.2, J1.2 (Pin_2), R1.1, R2.1, R3.1, R4.1, R5.1, U1.22 (GND), U1.8 (GND)
- new net ROW1: D1.2 (A), R1.2, SW1.1, SW10.1, SW11.1, SW2.1, SW3.1, SW4.1, SW5.1, SW6.1, SW7.1, SW8.1, SW9.1, U1.26 (PC3)
- new net ROW2: D2.2 (A), R2.2, SW12.1, SW13.1, SW14.1, SW15.1, SW16.1, SW17.1, SW18.1, SW19.1, SW20.1, SW21.1, SW22.1, U1.27 (PC4)
- new net ROW3: D3.2 (A), R3.2, SW23.1, SW24.1, SW25.1, SW26.1, SW27.1, SW28.1, SW29.1, SW30.1, SW31.1, SW32.1, SW33.1, U1.28 (PC5)
- new net ROW4: D4.2 (A), R4.2, SW34.1, SW35.1, SW36.1, SW37.1, SW38.1, SW39.1, SW40.1, SW41.1, SW42.1, U1.2 (PD0)
- new net Trigger: D1.1 (K), D2.1 (K), D3.1 (K), D4.1 (K), R5.2, U1.3 (PD1)
Other:
- added sheet 1 (2.kicad_sch)
